File: Boards/Rev B/Mini Flamingo Rev A.sch (KiCad schematic (older format))
At the start: 19 parts, among them J1 ISP_Header, J2 APA102C Out, J3 Batt Conn, SW1 Power Switch, U1 ATTINY85-20SU, U2 APA102C

Commit message: Mini Flamingo test code and Rev A fixes
Parts:
- S1: value Cycle -> Button 1
- S2: value Up -> Button 2
- S3: value Down -> Button 3
Connections:
- net ClockOut renamed APA102C_ClockOut
- net DataOut renamed APA102C_DataOut
- net MOSI/WS2812Data renamed MOSI/APA102C_Data
- net PIN2/SW2 renamed PIN2/Butt2
- net PIN3/SW3 renamed PIN3/Butt3
- net PIN6/SW1 renamed PIN6/Butt1
- net SCK/WS2812Clock renamed SCK/APA102C_Clock
Other:
- moved on the sheet: C2, D1, J2, J3, R1, R2, R3, R5, S1, S2, S3, SW1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
